Commit message: modified:   move_videoray/CMakeLists.txt 	new file:   move_videoray/graphics/videoray_robot.3ds 	modified:   move_videoray/graphics/videoray_robot.stl 	modified:   move_videoray/package.xml 	new file:   move_videoray/src/featureExtraction.cpp 	new file:   move_videoray/src/fullLimitFilter.cpp 	new file:   move_videoray/src/indicesFilter.cpp 	new file:   move_videoray/src/indicesFilter2.cpp 	new file:   move_videoray/src/kalman_filter.py 	new file:   move_videoray/src/kalman_filter.pyc 	new file:   move_videoray/src/limitFilter.cpp 	new file:   move_videoray/src/make_graph.py 	new file:   move_videoray/src/make_graph.pyc 	deleted:    move_videoray/src/move_filter02.py 	new file:   move_videoray/src/move_filtered02.py 	new file:   move_videoray/src/move_filtered03.py 	modified:   move_videoray/src/move_unfiltered.cpp 	modified:   move_videoray/src/move_unfiltered.py 	modified:   move_videoray/src/outlier_filter.py 	modified:   move_videoray/src/outlier_filter.pyc 	new file:   move_videoray/src/pointFilter.cpp 	new file:   move_videoray/src/smoothFilter.cpp 	new file:   move_videoray/src/voxelFilter.cpp 	modified:   move_videoray/videoray.urdf 	new file:   simLaunch.launch

File: move_videoray/videoray.urdf (robot description, URDF)
Before this commit: robot videoray, 2 links, 1 joints
Links:
- link body: geometry visual mesh filename=file:///home/nathaniel/simulation/src/ros-videoray-sim/move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
